Commit message: 이지컨트롤러 호환 (그리퍼)

File: urdf/my_robot.urdf (robot description, URDF)
Before this commit: robot assy2urdf, 13 links, 12 joints
Links:
- removed link XM,H-430_idler_Component5_v1_1
- removed link XM,H-430_idler_Component5_v1__1__1
- removed link XM,H-430_idler_Component5_v1__2__1
- removed link XM,H-430_idler_Component5_v1__3__1
- removed link XM,H-430_idler_Component5_v1__4__1
- removed link XM,H-430_idler_Component5_v1__5__1
- removed link piper_01_v1_1
- removed link piper_02_v1_1
- removed link piper_03_v1_1
- removed link piper_04_v2_1
- removed link piper_05_v1_1
- added link XM,H-430_idler_Component5_v2_1, mass 0.08200372676881872; collision mesh filename=package://gravity_compensation/meshes/XM,H-430_idler_Compon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 scale=0.001 0.001 0.001; visual mesh filename=package://gravity_compensation/meshes/XM,H-430_idler_Compon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 scale=0.001 0.001 0.001
- added link XM,H-430_idler_Component5_v2__1__1, mass 0.08200372676881872; collision mesh filename=package://gravity_compensation/meshes/XM,H-430_idler_Compon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 scale=0.001 0.001 0.001; visual mesh filename=package://gravity_compensation/meshes/XM,H-430_idler_Compon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 scale=0.001 0.001 0.001
- added link XM,H-430_idler_Component5_v2__2__1, mass 0.08200372676881872; collision mesh filename=package://gravity_compensation/meshes/XM,H-430_idler_Compon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 scale=0.001 0.001 0.001; visual mesh filename=package://gravity_compensation/meshes/XM,H-430_idler_Compon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 scale=0.001 0.001 0.001
- added link XM,H-430_idler_Component5_v2__3__1, mass 0.08200372676881872; collision mesh filename=package://gravity_compensation/meshes/XM,H-430_idler_Compon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 scale=0.001 0.001 0.001; visual mesh filename=package://gravity_compensation/meshes/XM,H-430_idler_Compon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 scale=0.001 0.001 0.001
- added link XM,H-430_idler_Component5_v2__4__1, mass 0.08200372676881872; collision mesh filename=package://gravity_compensation/meshes/XM,H-430_idler_Compon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 scale=0.001 0.001 0.001; visual mesh filename=package://gravity_compensation/meshes/XM,H-430_idler_Compon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 scale=0.001 0.001 0.001
- added link XM,H-430_idler_Component5_v2__5__1, mass 0.08200372676881872; collision mesh filename=package://gravity_compensation/meshes/XM,H-430_idler_Compon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 scale=0.001 0.001 0.001; visual mesh filename=package://gravity_compensation/meshes/XM,H-430_idler_Compon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 scale=0.001 0.001 0.001
- added link XM,H-430_idler_Component5_v2__6__1, mass 0.08200372676881872; collision mesh filename=package://gravity_compensation/meshes/XM,H-430_idler_Compon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 scale=0.001 0.001 0.001; visual mesh filename=package://gravity_compensation/meshes/XM,H-430_idler_Compon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 scale=0.001 0.001 0.001
- added link gripper_02_v1_1, mass 0.0156; collision mesh filename=package://gravity_compensation/meshes/gripper_02_v1_1.stl scale=0.001 0.001 0.001; visual mesh filename=package://gravity_compensation/meshes/gripper_02_v1_1.stl scale=0.001 0.001 0.001
- added link piper_01_v3_1, mass 0.01447; collision mesh filename=package://gravity_compensation/meshes/piper_01_v3_1.stl scale=0.001 0.001 0.001; visual mesh filename=package://gravity_compensation/meshes/piper_01_v3_1.stl scale=0.001 0.001 0.001
- added link piper_02_v2_1, mass 0.048; collision mesh filename=package://gravity_compensation/meshes/piper_02_v2_1.stl scale=0.001 0.001 0.001; visual mesh filename=package://gravity_compensation/meshes/piper_02_v2_1.stl scale=0.001 0.001 0.001
- added link piper_03_v2_1, mass 0.03698; collision mesh filename=package://gravity_compensation/meshes/piper_03_v2_1.stl scale=0.001 0.001 0.001; visual mesh filename=package://gravity_compensation/meshes/piper_03_v2_1.stl scale=0.001 0.001 0.001
- added link piper_04_v3_1, mass 0.0163; collision mesh filename=package://gravity_compensation/meshes/piper_04_v3_1.stl scale=0.001 0.001 0.001; visual mesh filename=package://gravity_compensation/meshes/piper_04_v3_1.stl scale=0.001 0.001 0.001
- added link piper_05_v2_1, mass 0.0163; collision mesh filename=package://gravity_compensation/meshes/piper_05_v2_1.stl scale=0.001 0.001 0.001; visual mesh filename=package://gravity_compensation/meshes/piper_05_v2_1.stl scale=0.001 0.001 0.001
Joints:
- added joint Revolute 14: type revolute, parent XM,H-430_idler_Component5_v2_1, child gripper_02_v1_1, origin xyz=0.019 0.0 0.03525 rpy=0 0 0, axis 1.0 0.0 0.0, limit lower=-0.785398 upper=0.785398 effort=100 velocity=100
- added joint Rigid 13: type fixed, parent gripper_01_v1_1, child XM,H-430_idler_Component5_v2_1, origin xyz=0.0 0.0 0.04 rpy=0 0 0
- joint Revolute 10: child piper_05_v1_1 -> piper_05_v2_1; limit lower=-1.57 upper=1.57 effort=10 velocity=3 -> lower=-1.570796 upper=1.570796 effort=100 velocity=100; parent XM,H-430_idler_Component5_v1__2__1 -> XM,H-430_idler_Component5_v2__3__1
- joint Revolute 12: limit lower=-1.57 upper=1.57 effort=10 velocity=3 -> lower=-1.570796 upper=1.570796 effort=100 velocity=100; parent XM,H-430_idler_Component5_v1__3__1 -> XM,H-430_idler_Component5_v2__5__1
- joint Revolute 2: child piper_01_v1_1 -> piper_01_v3_1; limit lower=-1.57 upper=1.57 effort=10 velocity=3 -> lower=-3.141593 upper=3.141593 effort=100 velocity=100; parent XM,H-430_idler_Component5_v1_1 -> XM,H-430_idler_Component5_v2__1__1
- joint Revolute 4: child piper_02_v1_1 -> piper_02_v2_1; limit lower=-3 upper=3 effort=10 velocity=3 -> lower=-3.14 upper=3.14 effort=100 velocity=100; parent XM,H-430_idler_Component5_v1__1__1 -> XM,H-430_idler_Component5_v2__6__1
- joint Revolute 6: child piper_03_v1_1 -> piper_03_v2_1; limit lower=-3 upper=3 effort=10 velocity=3 -> lower=-3.14 upper=3.14 effort=100 velocity=100; parent XM,H-430_idler_Component5_v1__5__1 -> XM,H-430_idler_Component5_v2__4__1
- joint Revolute 8: child piper_04_v2_1 -> piper_04_v3_1; limit lower=-1.57 upper=1.57 effort=10 velocity=3 -> lower=-1.570796 upper=1.570796 effort=100 velocity=100; parent XM,H-430_idler_Component5_v1__4__1 -> XM,H-430_idler_Component5_v2__2__1
- joint Rigid 1: child XM,H-430_idler_Component5_v1_1 -> XM,H-430_idler_Component5_v2__1__1
- joint Rigid 11: child XM,H-430_idler_Component5_v1__3__1 -> XM,H-430_idler_Component5_v2__5__1; parent piper_05_v1_1 -> piper_05_v2_1
- joint Rigid 3: child XM,H-430_idler_Component5_v1__1__1 -> XM,H-430_idler_Component5_v2__6__1; parent piper_01_v1_1 -> piper_01_v3_1
- joint Rigid 5: child XM,H-430_idler_Component5_v1__5__1 -> XM,H-430_idler_Component5_v2__4__1; parent piper_02_v1_1 -> piper_02_v2_1
- joint Rigid 7: child XM,H-430_idler_Component5_v1__4__1 -> XM,H-430_idler_Component5_v2__2__1; parent piper_03_v1_1 -> piper_03_v2_1
- joint Rigid 9: child XM,H-430_idler_Component5_v1__2__1 -> XM,H-430_idler_Component5_v2__3__1; parent piper_04_v2_1 -> piper_04_v3_1

Commit message: urdf 변경 및 tty 변경

File: urdf/my_robot.urdf (robot description, URDF)
Before this commit: robot assy2urdf, 15 links, 14 joints
Joints:
- removed joint Revolute 10
- removed joint Revolute 12
- removed joint Revolute 14
- removed joint Revolute 2
- removed joint Revolute 4
- removed joint Revolute 6
- removed joint Revolute 8
- added joint gripper: type revolute, parent XM,H-430_idler_Component5_v2_1, child gripper_02_v1_1, origin xyz=0.019 0.0 0.03525 rpy=0 0 0, axis 1.0 0.0 0.0, limit lower=-0.785398 upper=0.785398 effort=100 velocity=100
- added joint joint1: type revolute, parent XM,H-430_idler_Component5_v2__1__1, child piper_01_v3_1, origin xyz=-0.01425 0.004 0.025 rpy=0 0 0, axis 0.0 0.0 1.0, limit lower=-3.141593 upper=3.141593 effort=100 velocity=100
- added joint joint2: type revolute, parent XM,H-430_idler_Component5_v2__6__1, child piper_02_v2_1, origin xyz=-0.013 0.01425 0.028 rpy=0 0 0, axis -1.0 0.0 0.0, limit lower=-3.14 upper=3.14 effort=100 velocity=100
- added joint joint3: type revolute, parent XM,H-430_idler_Component5_v2__4__1, child piper_03_v2_1, origin xyz=0.013 0.01425 0.028 rpy=0 0 0, axis 1.0 0.0 -0.0, limit lower=-3.14 upper=3.14 effort=100 velocity=100
- added joint joint4: type revolute, parent XM,H-430_idler_Component5_v2__2__1, child piper_04_v3_1, origin xyz=-0.028 0.01425 0.025 rpy=0 0 0, axis -0.0 -0.0 1.0, limit lower=-1.570796 upper=1.570796 effort=100 velocity=100
- added joint joint5: type revolute, parent XM,H-430_idler_Component5_v2__3__1, child piper_05_v2_1, origin xyz=0.013 0.01425 0.028 rpy=0 0 0, axis 1.0 0.0 0.0, limit lower=-1.570796 upper=1.570796 effort=100 velocity=100
- added joint joint6: type revolute, parent XM,H-430_idler_Component5_v2__5__1, child gripper_01_v1_1, origin xyz=0.028 0.01425 0.013 rpy=0 0 0, axis -0.0 -0.0 1.0, limit lower=-1.570796 upper=1.570796 effort=100 velocity=100
